File: MAGFest2023SolderingClass/MAGFest2023SolderingClass.kicad_sch (KiCad schematic)
At the start: 18 parts, among them U1 ULN2002, U2 CH32V003a4m6

Commit message: Added ignore on gitignore, and SAO header
Parts:
- added J1: Conn_02x03_Odd_Even, Connector_PinHeader_2.54mm:PinHeader_2x03_P2.54mm_Vertical, symbol Connector_Generic:Conn_02x03_Odd_Even
Connections:
- net +3V3: now also J1.1 (Pin_1)
- net GND: now also J1.2 (Pin_2)
- net SWIO: now also J1.5 (Pin_5)
Changed lines of the file:
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@@
+    (stroke (width 0) (type default))
+  )
+  (wire (pts (xy 128.27 27.94) (xy 137.16 27.94))
     (stroke (width 0) (type default))
   )
@@
     (stroke (width 0) (type default))
   )
+  (wire (pts (xy 149.86 22.86) (xy 160.02 22.86))
+    (stroke (width 0) (type default))
+  )
   (wire (pts (xy 168.91 80.01) (xy 170.18 80.01))
     (stroke (width 0) (type default))
@@
     (stroke (width 0) (type default))
   )
+  (wire (pts (xy 137.16 22.86) (xy 128.27 22.86))
+    (stroke (width 0) (type default))
+  )
   (wire (pts (xy 154.94 62.23) (xy 154.94 45.72))
     (stroke (width 0) (type default))
@@
   (wire (pts (xy 153.67 80.01) (xy 163.83 80.01))
     (stroke (width 0) (type default))
+  )
+  (label "SWIO" (at 130.81 27.94 0) (fields_autoplaced)
+    (effects (font (size 1.27 1.27)) (justify left bottom))
   )
   (label "SWIO" (at 121.92 59.69 0) (fields_autoplaced)
@@
     )
   )
+  (symbol (lib_id "power:+3V3") (at 128.27 22.86 0) (unit 1)
+    (in_bom yes) (on_board yes) (dnp no) (fields_autoplaced)
+    (property "Reference" "#PWR06" (at 128.27 26.67 0)
+      (effects (font (size 1.27 1.27)) hide)
+    )
+    (property "Value" "+3V3" (at 128.27 17.78 0)
+      (effects (font (size 1.27 1.27)))
+    )
+    (property "Footprint" "" (at 128.27 22.86 0)
+      (effects (font (size 1.27 1.27)) hide)
+    )
+    (property "Datasheet" "" (at 128.27 22.86 0)
+      (effects (font (size 1.27 1.27)) hide)
+    )
+    (pin "1")
+    (instances
+      (project "MAGFest2023SolderingClass"
+        (path "/fa8e7198-2d30-4f64-8522-2f9b4d074595"
+          (reference "#PWR06") (unit 1)
+        )
+      )
+    )
+  )
   (symbol (lib_id "Device:C_Small") (at 165.1 48.26 0) (unit 1)
     (in_bom yes) (on_board yes) (dnp no) (fields_autoplaced)
@@
         )
       )
+    )
+  )
+  (symbol (lib_id "Connector_Generic:Conn_02x03_Odd_Even") (at 142.24 25.4 0) (unit 1)
+    (in_bom yes) (on_board yes) (dnp no) (fields_autoplaced)
+    (property "Reference" "J1" (at 143.51 16.51 0)
+      (effects (font (size 1.27 1.27)))
+    )
+    (property "Value" "Conn_02x03_Odd_Even" (at 143.51 19.05 0)
+      (effects (font (size 1.27 1.27)))
+    )
+    (property "Footprint" "Connector_PinHeader_2.54mm:PinHeader_2x03_P2.54mm_Vertical" (at 142.24 25.4 0)
+      (effects (font (size 1.27 1.27)) hide)
+    )
+    (property "Datasheet" "~" (at 142.24 25.4 0)
+      (effects (font (size 1.27 1.27)) hide)
+    )
+    (pin "5")
+    (pin "3")
+    (pin "6")
+    (pin "1")
+    (pin "2")
+    (pin "4")
+    (instances
+      (project "MAGFest2023SolderingClass"
+        (path "/fa8e7198-2d30-4f64-8522-2f9b4d074595"
+          (reference "J1") (unit 1)
+        )
+      )
+    )
+  )
+  (symbol (lib_id "power:GND") (at 160.02 22.86 0) (unit 1)
+    (in_bom yes) (on_board yes) (dnp no) (fields_autoplaced)
+    (property "Reference" "#PWR07" (at 160.02 29.21 0)
+      (effects (font (size 1.27 1.27)) hide)
+    )
+    (property "Value" "GND" (at 160.02 27.94 0)
+      (effects (font (size 1.27 1.27)))
+    )
+    (property "Footprint" "" (at 160.02 22.86 0)
+      (effects (font (size 1.27 1.27)) hide)
+    )
+    (property "Datasheet" "" (at 160.02 22.86 0)
+      (effects (font (size 1.27 1.27)) hide)
+    )
+    (pin "1")
+    (instances
+      (project "MAGFest2023SolderingClass"
+        (path "/fa8e7198-2d30-4f64-8522-2f9b4d074595"
+          (reference "#PWR07") (unit 1)
+        )
+      )
